File: PCB/kalam.kicad_pcb (KiCad board)
At the start: 2 copper layers, 246.5 x 75.1 mm, 116 parts, among them J1 Conn_01x04, SW1 SW_Push, U1 XC6206PxxxMR, U2 STM32F072CBTx

Commit message: rev1
Parts:
- added MX52: MX_SW_solder, PCM_marbastlib-mx:SW_MX_1u, F.Cu at (110.4, 79.5)
- added MX53: MX_SW_solder, PCM_marbastlib-mx:SW_MX_1u, F.Cu at (158.1, 79.5)
- added S7: 2.25, PCM_marbastlib-mx:STAB_MX_P_2.25u, F.Cu at (110.4, 79.5)
- added S8: 2.75, PCM_marbastlib-mx:STAB_MX_P_2.75u, F.Cu at (158.1, 79.5)
- moved D41 17.0 mm to (173.2, 80.2)
Routing:
- net col7: track 131.4 -> 146.8 mm
- net Net-(D41-A): track 5.67 -> 15.3 mm
- net Net-(D39-A): track 5.66 -> 8.04 mm
- net col4: track 185.7 -> 188.1 mm
- net row3: track 249.7 -> 249.1 mm
Other:
- board text added: "2"
- board text added: "2.25"
- board text added: "2.25u"
- board text added: "2.75"
- board text added: "2.75u"
- board text added: "6.25"
- board text added: "7"
