File: PCB/matrix.kicad_sch (KiCad schematic)
At the start: 101 parts

Commit message: rev1
Parts:
- added MX52, MX53: MX_SW_solder, PCM_marbastlib-mx:SW_MX_1u, symbol PCM_marbastlib-mx:MX_SW_solder
- added S7: 2.25, PCM_marbastlib-mx:STAB_MX_P_2.25u, symbol PCM_marbastlib-mx:MX_stab
- added S8: 2.75, PCM_marbastlib-mx:STAB_MX_P_2.75u, symbol PCM_marbastlib-mx:MX_stab
Connections:
- net col4: now also MX52.2
- net col7: now also MX53.1
- net at D39.2 (A), MX43.1: now also MX52.1
- net at D41.2 (A), MX46.1: now also MX53.2
